File: kicad/smart_gate_carrier/smart_gate_carrier.kicad_pcb (KiCad board)
At the start: 2 copper layers, 150 x 80 mm, 28 parts

Commit message: fix(kicad): use library mounting hole footprint to survive save/load
Previously add_outline_and_mounts.py built mount holes from a bare
pcbnew.FOOTPRINT(board) call without setting a library reference. KiCad 6
silently discarded them on save (no valid footprint identifier). Switched to
pcbnew.FootprintLoad(MountingHole, MountingHole_3.2mm_M3) which yields proper
library-backed footprints that persist through Save()/Load() cycles.

Co-Authored-By: Claude Opus 4.7 <noreply@anthropic.com>
Parts:
- removed the C_BULK at (110.0, 130.0)
- removed the C_LDOIN at (118.0, 155.0)
- removed the C_LDOOUT at (124.0, 155.0)
- removed the C_SVO at (230.0, 155.0)
- removed the D_REV at (125.0, 115.0)
- removed the J_BUCK at (125.0, 135.0)
- removed the J_BUZ at (230.0, 167.0)
- removed the J_ESP_L at (155.0, 140.0)
- removed the J_ESP_R at (178.0, 140.0)
- removed the J_EXP at (135.0, 170.0)
- removed the J_LCD at (230.0, 115.0)
- removed the J_PWR at (110.0, 115.0)
- removed the J_RFID at (205.0, 115.0)
- removed the J_SVO at (230.0, 140.0)
- removed the J_USR at (205.0, 145.0)
- removed the Q_BUZ at (205.0, 167.0)
- removed the R_BUZ at (213.0, 167.0)
- removed the R_SCL at (222.0, 132.0)
- removed the R_SDA at (222.0, 128.0)
- removed the U_LDO at (110.0, 155.0)
- added C_BULK: 100uF/25V, Capacitor_THT:CP_Radial_D8.0mm_P3.50mm, F.Cu at (110.0, 130.0)
- added C_LDOIN: 10uF, Capacitor_SMD:C_0805_2012Metric, F.Cu at (118.0, 155.0)
- added C_LDOOUT: 10uF, Capacitor_SMD:C_0805_2012Metric, F.Cu at (124.0, 155.0)
- added C_SVO: 470uF/16V, Capacitor_THT:CP_Radial_D10.0mm_P5.00mm, F.Cu at (230.0, 155.0)
- added D_REV: 1N5817, Diode_THT:D_DO-201AD_P15.24mm_Horizontal, F.Cu at (125.0, 115.0)
- added J_BUCK: Buck_12V_to_5V, Connector_PinHeader_2.54mm:PinHeader_1x04_P2.54mm_Vertical, F.Cu at (125.0, 135.0)
- added J_BUZ: Buzzer_Active, Connector_PinHeader_2.54mm:PinHeader_1x02_P2.54mm_Vertical, F.Cu at (230.0, 167.0)
- added J_ESP_L: DevKit_L, Connector_PinSocket_2.54mm:PinSocket_1x15_P2.54mm_Vertical, F.Cu at (155.0, 140.0)
- added J_ESP_R: DevKit_R, Connector_PinSocket_2.54mm:PinSocket_1x15_P2.54mm_Vertical, F.Cu at (178.0, 140.0)
- added J_EXP: Expansion, Connector_PinHeader_2.54mm:PinHeader_1x06_P2.54mm_Vertical, F.Cu at (135.0, 170.0)
- added J_LCD: LCD_20x4_I2C, Connector_PinHeader_2.54mm:PinHeader_1x04_P2.54mm_Vertical, F.Cu at (230.0, 115.0)
- added J_PWR: 12V_IN, Connector_BarrelJack:BarrelJack_Horizontal, F.Cu at (110.0, 115.0)
- added J_RFID: RC522, Connector_PinHeader_2.54mm:PinHeader_1x08_P2.54mm_Vertical, F.Cu at (205.0, 115.0)
- added J_SVO: Servo_SG90, Connector_PinHeader_2.54mm:PinHeader_1x03_P2.54mm_Vertical, F.Cu at (230.0, 140.0)
- added J_USR: HC-SR04, Connector_PinHeader_2.54mm:PinHeader_1x04_P2.54mm_Vertical, F.Cu at (205.0, 145.0)
- added Q_BUZ: 2N3904, Package_TO_SOT_THT:TO-92_Inline, F.Cu at (205.0, 167.0)
- added R_BUZ: 1k, Resistor_SMD:R_0805_2012Metric, F.Cu at (213.0, 167.0)
- added R_SCL: 4.7k, Resistor_SMD:R_0805_2012Metric, F.Cu at (222.0, 132.0)
- added R_SDA: 4.7k, Resistor_SMD:R_0805_2012Metric, F.Cu at (222.0, 128.0)
- added U_LDO: AMS1117-3.3, Package_TO_SOT_SMD:SOT-223-3_TabPin2, F.Cu at (110.0, 155.0)
- C_ESP_3V3_1, C_ESP_3V3_2: footprint C_0805_2012Metric -> Capacitor_SMD:C_0805_2012Metric
- H1, H2, H3, H4: value M3 -> MountingHole_3.2mm_M3; footprint (none) -> MountingHole_3.2mm_M3
- R_USR1, R_USR2: footprint R_0805_2012Metric -> Resistor_SMD:R_0805_2012Metric
